File: hardware/quad_hdmi_tx/hdmi_ch4.kicad_sch (KiCad schematic)
At the start: 30 parts, among them J4 HDMI_A, U41 ADV7513BSWZ, U42 TPD12S016PWR, U43 TLV1117LV18DCYR

Commit message: レイアウト rev B: 115 × 38 mm の細長い 6 層基板に再配置、ヘッダ配線を全数固定して DRC 未接続 0 / クリアランス違反 0
- 基板を HDMI 4 個分の横幅 (115 mm) × 縦 38 mm (横の 1/3) に変更、6 層 (F / GND / SIG1 / SIG2 / PWR / B)
- FPGA ヘッダ 2×40 を裏面に 2 本、長辺と平行に配置。ヘッダの列が各 ADV7513 の真下に来る
- J7/J8 のピン割り当てを配線経路に合わせて変更 (J7 = ADV 左辺の D13-23 + D1/D2/D4/D5/D10、J8 = 下辺の残り + CLK/DE/HS/VS/HPD/INT)
- RGB バス 30 本 × 4 ch、DDC/CEC/HPD、AVDD/PVDD の一部、FPGA_5V を gen_pcb.py で内層に固定配線 (交差しないレーン割り当て)
- 部品の再配置 (C01/C16/C20/R2/R4、左の 1V8 コンデンサ列を x=cx-10.3 へ)、1V8 の島の首を広げてプレーンの連続を確保
- FreeRouting 1.9 (-mp 24 -oit 1.0、約 10 分) で残りを配線: 配線 2010 本、ビア 634 個、TMDS はビアなし・ペア内長差 0.47 mm 以下
- ガーバー / ドリル / CPL / 各層 PDF と docs の画像を再生成、README と fpga_header_pinmap.csv を更新

Co-Authored-By: Claude Fable 5.1 <noreply@anthropic.com>
Claude-Session: https://claude.ai/code/session_01JGo25NCpKCcdkj7JC5mDdQ
Parts:
- U41: footprint Package_QFP:LQFP-64-1EP_10x10mm_P0.5mm_EP5x5mm_ThermalVias -> Package_QFP:LQFP-64-1EP_10x10mm_P0.5mm_EP5x5mm
Changed lines of the file:
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@@
     (property "Reference" "U41" (at 122.54 127.46 0) (effects (font (size 1.27 1.27)) (justify left)))
     (property "Value" "ADV7513BSWZ" (at 122.54 130 0) (effects (font (size 1.27 1.27)) (justify left)))
-    (property "Footprint" "Package_QFP:LQFP-64-1EP_10x10mm_P0.5mm_EP5x5mm_ThermalVias" (at 120 130 0)
+    (property "Footprint" "Package_QFP:LQFP-64-1EP_10x10mm_P0.5mm_EP5x5mm" (at 120 130 0)
       (effects (font (size 1.27 1.27)) hide))
     (property "Datasheet" "~" (at 120 130 0) (effects (font (size 1.27 1.27)) hide))
