File: hardware/quad_hdmi_tx/power.kicad_sch (KiCad schematic)
At the start: 20 parts, among them J5 USB-C 5V in, J6 5V ALT IN, U5 AP63203WU

Commit message: レイアウト: 囲われたパッドへのアクセスビア、連続 GND ピンの数珠つなぎ、5V_OUT 事前配線、事前配線 DRC クリーン
Co-Authored-By: Claude Fable 5.1 <noreply@anthropic.com>
Claude-Session: https://claude.ai/code/session_01JGo25NCpKCcdkj7JC5mDdQ
Parts:
- H1, H2, H3, H4: footprint MountingHole:MountingHole_3.2mm_M3 -> MountingHole:MountingHole_3.2mm
Changed lines of the file:
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@@
     (property "Reference" "H1" (at 32.54 227.46 0) (effects (font (size 1.27 1.27)) (justify left)))
     (property "Value" "M3" (at 32.54 230 0) (effects (font (size 1.27 1.27)) (justify left)))
-    (property "Footprint" "MountingHole:MountingHole_3.2mm_M3" (at 30 230 0)
+    (property "Footprint" "MountingHole:MountingHole_3.2mm" (at 30 230 0)
       (effects (font (size 1.27 1.27)) hide))
     (property "Datasheet" "~" (at 30 230 0) (effects (font (size 1.27 1.27)) hide))
@@
     (property "Reference" "H2" (at 47.54 227.46 0) (effects (font (size 1.27 1.27)) (justify left)))
     (property "Value" "M3" (at 47.54 230 0) (effects (font (size 1.27 1.27)) (justify left)))
-    (property "Footprint" "MountingHole:MountingHole_3.2mm_M3" (at 45 230 0)
+    (property "Footprint" "MountingHole:MountingHole_3.2mm" (at 45 230 0)
       (effects (font (size 1.27 1.27)) hide))
     (property "Datasheet" "~" (at 45 230 0) (effects (font (size 1.27 1.27)) hide))
@@
     (property "Reference" "H3" (at 62.54 227.46 0) (effects (font (size 1.27 1.27)) (justify left)))
     (property "Value" "M3" (at 62.54 230 0) (effects (font (size 1.27 1.27)) (justify left)))
-    (property "Footprint" "MountingHole:MountingHole_3.2mm_M3" (at 60 230 0)
+    (property "Footprint" "MountingHole:MountingHole_3.2mm" (at 60 230 0)
       (effects (font (size 1.27 1.27)) hide))
     (property "Datasheet" "~" (at 60 230 0) (effects (font (size 1.27 1.27)) hide))
@@
     (property "Reference" "H4" (at 77.54 227.46 0) (effects (font (size 1.27 1.27)) (justify left)))
     (property "Value" "M3" (at 77.54 230 0) (effects (font (size 1.27 1.27)) (justify left)))
-    (property "Footprint" "MountingHole:MountingHole_3.2mm_M3" (at 75 230 0)
+    (property "Footprint" "MountingHole:MountingHole_3.2mm" (at 75 230 0)
       (effects (font (size 1.27 1.27)) hide))
     (property "Datasheet" "~" (at 75 230 0) (effects (font (size 1.27 1.27)) hide))
